Commit message: creating objects with xarco macro

File: src/ur_description/urdf/rrbot_grip.xacro (robot description, xacro)
@@ -3,11 +3,12 @@
 <robot xmlns:xacro="http://ros.org/wiki/xacro">
 <xacro:property name="dist" value="1.0" /> <!-- Link 3 -->
-<xacro:property name="mass_obj" value="1" /> <!-- arbitrary value for mass -->
-<xacro:property name="width" value="0.2" /> <!-- Square dimensions (widthxwidth) of beams -->
-<xacro:property name="height" value=".4" /> <!-- Link 1 -->
+<!--xacro:property name="mass_obj" value="1" /--> <!-- arbitrary value for mass -->
+<!--xacro:property name="width" value="0.2" /--> <!-- Square dimensions (widthxwidth) of beams -->
+<!--xacro:property name="height" value=".4" /--> <!-- Link 1 -->
   <!-- Constants for robot dimensions -->
-<link name="box">
+<xacro:macro name="obj_box" params="name1 name2 width height mass_obj *origin">
+<link name="${name1}">
     <collision>
-      <origin xyz="-1 ${dist} ${height/2}" rpy="0 0 0"/>
+      <xacro:insert_block name="origin" />
       <geometry>
 	<box size="${width} ${width} ${height}"/>
@@ -15,5 +16,5 @@
     </collision>
    <visual>
-      <origin xyz="-1 ${dist} ${height/2}" rpy="0 0 0"/>
+      <xacro:insert_block name="origin" />
       <geometry>
 	<box size="${width} ${width} ${height}"/>
@@ -22,5 +23,5 @@
     </visual>
     <inertial>
-      <origin xyz="-1 ${2.0} 0.5" rpy="0 0 0"/>
+      <xacro:insert_block name="origin" />
       <mass value="${mass_obj}"/>
       <inertia
@@ -30,6 +31,5 @@
     </inertial>
   </link>
-  <!--xarco:macro name="grip_plam" params="prefix"-->
-<link name="box1">
+<link name="${name2}">
     <!--collision>
       <origin xyz="-1 ${dist} .05" rpy="0 0 0"/>
@@ -49,38 +49,27 @@
       <mass value="${mass_obj}"/>
       <inertia
-	  ixx="${mass_obj / 12.0 * (width*width + height*height)}" ixy="0.0" ixz="0.0"
-	  iyy="${mass_obj / 12.0 * (height*height + width*width)}" iyz="0.0"
-	  izz="${mass_obj / 12.0 * (width*width + width*width)}"/>
+	  ixx="${0 / 12.0 * (width*width + height*height)}" ixy="0.0" ixz="0.0"
+	  iyy="${0 / 12.0 * (height*height + width*width)}" iyz="0.0"
+	  izz="${0 / 12.0 * (width*width + width*width)}"/>
     </inertial>
   </link>
-  <!--joint name="fixed" type="fixed">
-    <parent link="world"/>
-    <child link="box1"/>
-  </joint-->
-  <!--joint name="linx_joint" type="prismatic">
-    <parent link="world"/>
-    <child link="box"/>
+  <joint name="${name1}_linx_joint" type="prismatic">
+    <parent link="${prefix}world"/>
+    <child link="_${name1}"/>
     <axis xyz="1 0 0"/>
     <limit lower="0" upper="5" effort="1000" velocity="1.0"/>
   </joint>
-  </xarco:macro>
-  <joint name="joint_plam" type="prismatic">
-    <parent link="world"/>
-    <child link="box"/>
-    <axis xyz="1 0 0"/>
+  <joint name="${name1}_liny_joint" type="prismatic">
+    <parent link="_${name1}"/>
+    <child link="${name1}"/>
+    <axis xyz="0 1 0"/>
     <limit lower="0" upper="5" effort="1000" velocity="1.0"/>
-  </joint-->
-  <!--joint name="liny_joint" type="prismatic">
-    <parent link="link1"/>
-    <child link="box"/>
-    <axis xyz="0 1 0"/>
-    <limit lower="0" upper="5" effort="1000" velocity="0.2"/>
-  </joint-->
-<transmission name="lx_transmission">
+   </joint>
+<transmission name="${name1}_lx_transmission">
     <type>transmission_interface/SimpleTransmission</type>
-    <joint name="linx_joint">
+    <joint name="${name1}_linx_joint">
       <hardwareInterface>hardware_interface/VelocityJointInterface </hardwareInterface>
     </joint>
-    <actuator name="lx_motor">
+    <actuator name="${name1}_lx_motor">
       <hardwareInterface>hardware_interface/VelocityJointInterface </hardwareInterface>
       <mechanicalReduction>1</mechanicalReduction>
@@ -97,13 +86,20 @@
     </actuator>
 </transmission-->
-<transmission name="ly_transmission">
+<transmission name="${name1}_ly_transmission">
     <type>transmission_interface/SimpleTransmission</type>
-    <joint name="liny_joint">
+    <joint name="${name1}_liny_joint">
       <hardwareInterface>hardware_interface/VelocityJointInterface </hardwareInterface>
     </joint>
-    <actuator name="ly_motor">
+    <actuator name="${name1}_ly_motor">
       <hardwareInterface>hardware_interface/VelocityJointInterface </hardwareInterface>
       <mechanicalReduction>1</mechanicalReduction>
     </actuator>
 </transmission>
+</xacro:macro>
+<xacro:obj_box name1="box1" name2="_box1" width=".2" height=".4" mass_obj="1">
+        <origin xyz="-1 1 0.2" rpy="0 0 0"/>
+</xacro:obj_box>
+<xacro:obj_box name1="box2" name2="_box2" width=".2" height=".4" mass_obj="1">
+        <origin xyz="1 1 0.2" rpy="0 0 0"/>
+</xacro:obj_box>
 </robot>

File: src/ur_description/urdf/ur10.urdf.xacro (robot description, xacro)
@@ -60,16 +60,4 @@
     <xacro:property name="wrist_3_length" value="${d6}" />
     <xacro:include filename="$(find ur_description)/urdf/rrbot_grip.xacro" />
-    <joint name="linx_joint" type="prismatic">
-    <parent link="${prefix}world"/>
-    <child link="box1"/>
-    <axis xyz="1 0 0"/>
-    <limit lower="0" upper="5" effort="1000" velocity="1.0"/>
-    </joint>
-    <joint name="liny_joint" type="prismatic">
-    <parent link="box1"/>
-    <child link="box"/>
-    <axis xyz="0 1 0"/>
-    <limit lower="0" upper="5" effort="1000" velocity="0.2"/>
-    </joint>
     <link name="${prefix}base_link" >
       <visual>
